File: esp-bldc-foc.kicad_pcb (KiCad board)
At the start: 4 copper layers, 66 x 66 mm, 96 parts, among them IC1 ESP32-S3FN8, IC2 LY68L6400SLIT, IC3 AS5600-ASOM, J1 USB_C_Receptacle_USB2.0, J10 UART, J3 I2C ENCODER, J6 Conn_01x02_Female, J7 A, J8 B, J9 C, Q1 BUK7M9R9-60EX, Q10 BUK7M9R9-60EX, Q11 BUK7M9R9-60EX, Q12 BUK7M9R9-60EX, Q2 BUK7M9R9-60EX, Q3 BUK7M9R9-60EX, Q4 BUK7M9R9-60EX, Q5 BUK7M9R9-60EX, Q6 BUK7M9R9-60EX, Q7 BUK7M9R9-60EX, Q8 BUK7M9R9-60EX, Q9 BUK7M9R9-60EX, SW1 SW_SPST, SW2 SW_SPST, U1 ADP7182AUJZ-3.3, U2 DRV8353SMRTAT, U5 LMR36510ADDA, Y1 40MHz

Commit message: Adding step
Parts:
- removed TP1, TP2: TestPoint, TestPoint:TestPoint_Pad_D2.5mm
- R19, R22, R8: value 500u -> 0.002R; footprint Resistor_SMD:R_2010_5025Metric -> Resistor_SMD:R_2816_7142Metric
- moved NT5 6.22 mm to (168.2, 112.3), turned to 0 degrees
- moved C21 3.19 mm to (151.3, 99.0)
- moved NT7 2.74 mm to (157.4, 77.9)
- moved R8 1.94 mm to (152.2, 104.3)
- moved R19 1.56 mm to (169.7, 115.5)
- moved R22 1.54 mm to (161.4, 80.4)
- moved C23 1.25 mm to (158.3, 82.6)
- moved NT3 0.61 mm to (149.4, 105.3)
Routing:
- net /Power_stage/SP2: track 48.5 -> 41.2 mm
- net /Power_stage/SP3: track 13.4 -> 16.0 mm
- net /Power_stage/SN1: track 22.1 -> 24.0 mm
- net /Power_stage/SN3: track 14.4 -> 13.2 mm
- net /Power_stage/SP1: track 27.9 -> 27.3 mm
- net GND: track 78.5 -> 78.7 mm, vias 276 -> 269
- net VBUS: vias 391 -> 365
- net Net-(AE1-Pad2): vias 4 -> 0
- net +3.3V: vias 133 -> 136
- net (no net): vias 5 -> 0
