File: Power_reg.kicad_sch (KiCad schematic)
At the start: 31 parts, among them J6 Conn_01x02_Female, U4 LMR36510ADDA, U5 LMR36510ADDA

Commit message: Routing done
Parts:
- removed C33, C35: 220nF, Capacitor_SMD:C_0402_1005Metric, symbol Device:C
- removed C37: 1uF, Capacitor_SMD:C_0402_1005Metric, symbol Device:C
- removed C39: 100nF, Capacitor_SMD:C_0402_1005Metric, symbol Device:C
- removed C41: 10pF, Capacitor_SMD:C_0402_1005Metric, symbol Device:C
- removed C43: 47uF, Capacitor_SMD:C_1206_3216Metric, symbol Device:C
- removed D5: D, Diode_SMD:D_0805_2012Metric, symbol Device:D
- removed L3: 22uH, Inductor_SMD:L_Bourns-SRN4018, symbol Device:L
- removed R23: 100K, Resistor_SMD:R_0402_1005Metric, symbol Device:R
- removed R24: 24.9K, Resistor_SMD:R_0402_1005Metric, symbol Device:R
- removed U4: LMR36510ADDA, Package_SO:Texas_HTSOP-8-1EP_3.9x4.9mm_P1.27mm_EP2.95x4.9mm_Mask2.4x3.1mm_ThermalVias, symbol Regulator_Switching:LMR36510ADDA
Connections:
- no-connect marks 2 -> 1
